File: adc_ad7794/adc_ad7794.sch (KiCad schematic (older format))
At the start: 34 parts, among them U1 AD7794

Commit message: Add files via upload
Parts:
- added RJUMPER1: 0, Resistor_SMD:R_0805_2012Metric_Pad1.15x1.40mm_HandSolder, symbol Device:R
- CA1, CD1: footprint (none) -> Capacitor_Tantalum_SMD:CP_EIA-6032-20_AVX-F_Pad2.25x2.35mm_HandSolder
- CA2, CD2: footprint (none) -> Capacitor_SMD:C_1206_3216Metric_Pad1.42x1.75mm_HandSolder
- D1, D2, D3: footprint (none) -> Diode_SMD:D_1210_3225Metric_Pad1.42x2.65mm_HandSolder
- D4: renamed from D?; footprint (none) -> Diode_SMD:D_1210_3225Metric_Pad1.42x2.65mm_HandSolder
- JCLK1: renamed from JCLK; footprint (none) -> TestPoint:TestPoint_Pad_D2.0mm
- JDIG1: renamed from JDIG; footprint (none) -> TerminalBlock_Altech:Altech_AK300_1x04_P5.00mm_45-Degree
- JIN1: renamed from JIN; footprint (none) -> TerminalBlock_Altech:Altech_AK300_1x12_P5.00mm_45-Degree
- JPOWER1: renamed from JPOWER; footprint (none) -> TerminalBlock_Altech:Altech_AK300_1x03_P5.00mm_45-Degree
- JPSW1: renamed from JPSW; footprint (none) -> TestPoint:TestPoint_Pad_D2.0mm
- JREFNEG1: renamed from JREFNEG; footprint (none) -> TestPoint:TestPoint_Pad_D2.0mm
- JREFPOS1: renamed from JREFPOS; footprint (none) -> TestPoint:TestPoint_Pad_D2.0mm
- L1, L2: value INDUCTOR -> ferrita; footprint (none) -> Inductor_SMD:L_1206_3216Metric_Pad1.42x1.75mm_HandSolder
- R11, R12, R21, R22, R31, R32, R41, R42, R51, R52, R61, R62, RUP1, RUP2, RUP3, RUP4: footprint (none) -> Resistor_SMD:R_0805_2012Metric_Pad1.15x1.40mm_HandSolder
Connections:
- net GNDA: now also RJUMPER1.2; no longer CD1.2, CD2.2, D3.2 (A), D4.2 (A), JPOWER1.3 (Pin_3)
- net at R11.1: now also U1.5 (AIN6+/P1); no longer U1.7 (AIN1+)
- net at R12.1: now also U1.6 (AIN6-/P2); no longer U1.8 (AIN1-)
- net POWER_DIG: now reaches D1.2 (A), JPOWER1.1 (Pin_1)
- net POWER_5V: now reaches D2.2 (A), JPOWER1.2 (Pin_2)
- net DOUT: now reaches JDIG1.1 (Pin_1), RUP1.2, U1.23 (DOUT/~RDY)
- net DIN: now reaches JDIG1.2 (Pin_2), RUP2.2, U1.24 (DIN)
- net CS: now reaches JDIG1.3 (Pin_3), RUP3.2, U1.3 (~CS)
- net SCLK: now reaches JDIG1.4 (Pin_4), RUP4.2, U1.1 (SCLK)
- net at R22.1: now also U1.8 (AIN1-); no longer U1.10 (AIN2-)
- net at R21.1: now also U1.7 (AIN1+); no longer U1.9 (AIN2+)
- net at R31.1: now also U1.9 (AIN2+); no longer U1.11 (AIN3+)
- net at R32.1: now also U1.10 (AIN2-); no longer U1.12 (AIN3-)
- net at R41.1: now also U1.11 (AIN3+); no longer U1.17 (AIN4+/REFIN2+)
- net at R42.1: now also U1.12 (AIN3-); no longer U1.18 (AIN4-/REFIN2-)
- net at R61.1: now also U1.17 (AIN4+/REFIN2+); no longer U1.5 (AIN6+/P1)
- net at R62.1: now also U1.18 (AIN4-/REFIN2-); no longer U1.6 (AIN6-/P2)
- new net GNDD: CD1.2, CD2.2, D3.2 (A), D4.2 (A), JPOWER1.3 (Pin_3), RJUMPER1.1
Other:
- moved on the sheet: JIN1, R11, R12, R21, R22, R31, R32, R41, R42, R51, R52, R61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
